File: electronics_design/kicad/car_inputs.kicad_sch (KiCad schematic)
At the start: 23 parts, among them J1 Conn_01x05_PinConn_Header_JST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, J2 Conn_Header_JST_PH_1x04_P2mm_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, J3 Conn_Header_JST_PH_1x04_P2mm_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, J4 Conn_Header_JST_PH_1x04_P2mm_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, J5 Conn_Header_JST_PH_1x03_P2mm_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, J6 Conn_Header_JST_PH_1x03_P2mm_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, M1 Module_XIAO-RP2040

Commit message: Replace 5V encoder power with 3V3
Connections:
- net +3V3: now also J1.1 (Pin_1)
- net +5V: no longer J1.1 (Pin_1)
Changed lines of the file:
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@@
 	)
 	(symbol
-		(lib_id "power:+5V")
+		(lib_id "power:+3V3")
 		(at 64.77 24.13 270)
 		(unit 1)
@@
 			)
 		)
-		(property "Value" "+5V"
+		(property "Value" "+3V3"
 			(at 68.58 24.1299 90)
 			(show_name no)
@@
 			)
 		)
-		(property "Description" "Power symbol creates a global label with name \"+5V\""
+		(property "Description" "Power symbol creates a global label with name \"+3V3\""
 			(at 64.77 24.13 0)
 			(hide yes)
